Commit message: ADD New macros for the new sensor plugins implementations from uuv_simulator
Signed-off-by: Musa Morena Marcusso Manhaes <Musa.Marcusso@de.bosch.com>

File: rexrov2_description/robots/rexrov2_default.xacro (robot description, xacro)
@@ -16,9 +16,13 @@
   <xacro:arg name="namespace" default="rexrov2"/>
   <xacro:arg name="use_simplified_mesh" default="false"/>
+  <xacro:arg name="inertial_reference_frame" default="world"/>
   <!-- Include the ROV macro file -->
   <xacro:include filename="$(find rexrov2_description)/urdf/rexrov2_base.xacro"/>
   <xacro:include filename="$(find rexrov2_description)/urdf/rexrov2.gazebo.xacro"/>
   <!-- Create the rexrov2 -->
-  <xacro:rexrov2_base namespace="$(arg namespace)" use_simplified_mesh="$(arg use_simplified_mesh)">
+  <xacro:rexrov2_base
+    namespace="$(arg namespace)"
+    use_simplified_mesh="$(arg use_simplified_mesh)"
+    inertial_reference_frame="$(arg inertial_reference_frame)">
     <!--
       The underwater object plugin is given as an input block parameter to

File: rexrov2_description/robots/rexrov2_oberon4.xacro (robot description, xacro)
@@ -16,4 +16,5 @@
   <xacro:arg name="namespace" default="rexrov2"/>
   <xacro:arg name="use_simplified_mesh" default="false"/>
+  <xacro:arg name="inertial_reference_frame" default="world"/>
   <!-- Include the ROV macro file -->
   <xacro:include filename="$(find rexrov2_description)/urdf/rexrov2_base.xacro"/>
@@ -21,5 +22,8 @@
   <xacro:include filename="$(find oberon4_description)/robots/oberon4_default.xacro" />
   <!-- Create the ROV -->
-  <xacro:rexrov2_base namespace="$(arg namespace)" use_simplified_mesh="$(arg use_simplified_mesh)">
+  <xacro:rexrov2_base
+    namespace="$(arg namespace)"
+    use_simplified_mesh="$(arg use_simplified_mesh)"
+    inertial_reference_frame="$(arg inertial_reference_frame)">
     <!-- The underwater object plugin is given as an input block parameter to
      allow the addition of external models of manipulator units -->

File: rexrov2_description/robots/rexrov2_oberon7.xacro (robot description, xacro)
@@ -16,4 +16,5 @@
   <xacro:arg name="namespace" default="rexrov2"/>
   <xacro:arg name="use_simplified_mesh" default="false"/>
+  <xacro:arg name="inertial_reference_frame" default="world"/>
   <!-- Include the ROV macro file -->
   <xacro:include filename="$(find rexrov2_description)/urdf/rexrov2_base.xacro"/>
@@ -21,5 +22,8 @@
   <xacro:include filename="$(find oberon7_description)/robots/oberon7_default.xacro" />
   <!-- Create the ROV -->
-  <xacro:rexrov2_base namespace="$(arg namespace)" use_simplified_mesh="$(arg use_simplified_mesh)">
+  <xacro:rexrov2_base
+    namespace="$(arg namespace)"
+    use_simplified_mesh="$(arg use_simplified_mesh)"
+    inertial_reference_frame="$(arg inertial_reference_frame)">
     <!-- The underwater object plugin is given as an input block parameter to
      allow the addition of external models of manipulator units -->

File: rexrov2_description/robots/rexrov2_oberon_arms.xacro (robot description, xacro)
@@ -16,4 +16,5 @@
   <xacro:arg name="namespace" default="rexrov2"/>
   <xacro:arg name="use_simplified_mesh" default="false"/>
+  <xacro:arg name="inertial_reference_frame" default="world"/>
   <!-- Include the ROV macro file -->
   <xacro:include filename="$(find rexrov2_description)/urdf/rexrov2_base.xacro"/>
@@ -22,5 +23,8 @@
   <xacro:include filename="$(find oberon7_description)/robots/oberon7_default.xacro" />
   <!-- Create the ROV -->
-  <xacro:rexrov2_base namespace="$(arg namespace)" use_simplified_mesh="$(arg use_simplified_mesh)">
+  <xacro:rexrov2_base
+    namespace="$(arg namespace)"
+    use_simplified_mesh="$(arg use_simplified_mesh)"
+    inertial_reference_frame="$(arg inertial_reference_frame)">
     <!-- The underwater object plugin is given as an input block parameter to
      allow the addition of external models of manipulator units -->

File: rexrov2_description/urdf/rexrov2_base.xacro (robot description, xacro)
@@ -14,5 +14,5 @@
 <robot xmlns:xacro="http://www.ros.org/wiki/xacro" >
   <xacro:include filename="$(find uuv_descriptions)/models/common/urdf/common.urdf.xacro"/>
-  <xacro:include filename="$(find uuv_sensor_plugins_ros)/urdf/sensor_snippets.xacro"/>
+  <xacro:include filename="$(find uuv_sensor_ros_plugins)/urdf/sensor_snippets.xacro"/>
   <xacro:include filename="$(find rexrov2_description)/urdf/rexrov2_snippets.xacro" />
   <xacro:include filename="$(find uuv_gazebo_ros_plugins)/urdf/snippets.xacro"/>
@@ -21,10 +21,11 @@
   <!-- Mass, see p.28 in Berg2012 -->
   <xacro:property name="mass" value="1862.87"/>
-  <xacro:macro name="rexrov2_base" params="namespace *gazebo use_simplified_mesh">
+  <xacro:macro name="rexrov2_base"
+    params="namespace *gazebo use_simplified_mesh inertial_reference_frame">
     <!-- Defining base link according to ROS conventions: x forward, z up -->
     <link name="${namespace}/base_link">
       <inertial>
         <mass value="${mass}"/>
-        <origin xyz="0 0 0"/>
+        <origin xyz="0 0 0" rpy="0 0 0"/>
         <inertia ixx="525.39" ixy="1.44" ixz="33.41" iyy="794.20" iyz="2.6" izz="691.23"/>
       </inertial>

File: rexrov2_description/urdf/rexrov2_sensors.xacro (robot description, xacro)
@@ -14,7 +14,12 @@
 <robot xmlns:xacro="http://www.ros.org/wiki/xacro" >
   <!-- DVL  -->
-  <xacro:default_dvl namespace="${namespace}" parent_link="${namespace}/base_link">
+  <xacro:default_dvl_macro
+    namespace="${namespace}"
+    parent_link="${namespace}/base_link"
+    inertial_reference_frame="${inertial_reference_frame}">
     <origin xyz="0.294307 0.468494 -0.68" rpy="0 ${0.5*pi} 0"/>
-  </xacro:default_dvl>
+  </xacro:default_dvl_macro>
+  <!-- Magnetometer  -->
+  <xacro:default_magnetometer namespace="${namespace}" parent_link="${namespace}/base_link"/>
   <!-- RPT  -->
   <xacro:default_rpt namespace="${namespace}" parent_link="${namespace}/base_link">
@@ -22,19 +27,31 @@
   </xacro:default_rpt>
   <!-- Pressure  -->
-  <xacro:default_pressure namespace="${namespace}" parent_link="${namespace}/base_link">
+  <xacro:default_pressure_macro namespace="${namespace}" parent_link="${namespace}/base_link">
     <origin xyz="-1.32 0.5 0.85" rpy="0 0 0"/>
-  </xacro:default_pressure>
+  </xacro:default_pressure_macro>
   <!-- IMU  -->
-  <xacro:default_imu namespace="${namespace}" parent_link="${namespace}/base_link">
+  <xacro:default_imu_macro
+    namespace="${namespace}"
+    parent_link="${namespace}/base_link"
+    inertial_reference_frame="${inertial_reference_frame}">
     <origin xyz="0 0 0" rpy="0 0 0"/>
-  </xacro:default_imu>
+  </xacro:default_imu_macro>
   <!-- Mount a camera -->
-  <xacro:default_camera namespace="${namespace}" parent_link="${namespace}/base_link" suffix="">
+  <xacro:default_camera
+    namespace="${namespace}"
+    parent_link="${namespace}/base_link"
+    suffix="">
     <origin xyz="1.15 0 0.4" rpy="0 0.6 0"/>
   </xacro:default_camera>
-  <xacro:default_camera namespace="${namespace}" parent_link="${namespace}/base_link" suffix="right">
+  <xacro:default_camera
+    namespace="${namespace}"
+    parent_link="${namespace}/base_link"
+    suffix="right">
     <origin xyz="1.15 -0.63 0.4" rpy="0 0.6 0.4"/>
   </xacro:default_camera>
-  <xacro:default_camera namespace="${namespace}" parent_link="${namespace}/base_link" suffix="left">
+  <xacro:default_camera
+    namespace="${namespace}"
+    parent_link="${namespace}/base_link"
+    suffix="left">
     <origin xyz="1.15 0.63 0.4" rpy="0 0.6 -0.4"/>
   </xacro:default_camera>
@@ -42,8 +59,14 @@
   <xacro:default_gps namespace="${namespace}" parent_link="${namespace}/base_link" />
   <!-- Mount a Pose 3D sensor. -->
-  <xacro:default_pose_3d namespace="${namespace}" parent_link="${namespace}/base_link" />
+  <xacro:default_pose_3d_macro
+    namespace="${namespace}"
+    parent_link="${namespace}/base_link"
+    inertial_reference_frame="${inertial_reference_frame}" />
   <!-- Mount chemical particle concentration sensor -->
-  <xacro:default_chemical_concentration_sensor namespace="${namespace}" parent_link="${namespace}/base_link">
+  <xacro:default_chemical_concentration_sensor_macro
+    namespace="${namespace}"
+    parent_link="${namespace}/base_link"
+    inertial_reference_frame="${inertial_reference_frame}">
     <origin xyz="0 0 0" rpy="0 0 0"/>
-  </xacro:default_chemical_concentration_sensor>
+  </xacro:default_chemical_concentration_sensor_macro>
 </robot>
